Commit message: Altering material name due to clash

File: kmriiwa_description/urdf/iiwa14/materials.xacro (robot description, xacro)
@@ -28,5 +28,5 @@
     <color rgba="1.0 1.0 1.0 1.0"/>
   </material>
-  <material name="aluminum">
+  <material name="iiwa_aluminum">
       <color rgba="0.5 0.5 0.5 1"/>
   </material>
